File: hardware/ProMini-Node-v1.0-50x50.kicad_pcb (KiCad board)
At the start: 2 copper layers, 45 x 50 mm, 69 parts, among them P1 Ant_SMA, P2 Power Input, P3 CONN_1, P4 CONN_2, P5 CONN_3, P6 CONN_4, P7 Ant, P8 Ant_uFL, P9 CONN_4, Q1 BSS84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

Commit message: Update renders, added BOM
Parts:
- removed G*** (x2): LOGO, Custom_Logos:ttn_logo-3
- removed REF**: OSHW-Logo2_7.3x6mm_SilkScreen, Symbol:OSHW-Logo2_7.3x6mm_SilkScreen
- C1: value C -> 100nF
- R1: value 100k -> 100K
- R2: value R -> 470K
- R3: value R -> 100K
