File: hardware/ProMini-Node-v1.0-50x50.kicad_sch (KiCad schematic)
At the start: 17 parts, among them P1 Ant_SMA, P2 Power Input, P3 CONN_1, P4 CONN_2, P5 CONN_3, P6 CONN_4, P7 Ant, P8 Ant_uFL, P9 CONN_4, Q1 BSS84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

Commit message: Sch update
Parts:
- C1: value C -> 100nF
- R1: value 100k -> 100K
- R2: value R -> 470K
- R3: value R -> 100K
Other:
- note added: "Min: 3.6V Max: 10V"
- moved on the sheet: C1, JP1, P1, P2, P7, P8, P9, Q1, R1, R2, R3, U1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

Commit message: example firmware update
Other:
- note added: "Pro RFM9x Mini ----------- VCC 3.3V GND GND D2 DIO0 D3 DIO1 D7 DIO2 D6 DIO5 D5 RESET D10-SS NSS D11-MOSI MOSI D12-MISO MISO D13-CLK SCK"
- note removed: "Pro RFM9x Mini ----------- VCC 3.3V GND GND D2 DIO0 D3 DIO1 D7 DIO2 D6 DIO5 D5 RESET D10-SS NSS MOSI MOSI MISO MISO CLK SCK"
Changed lines of the file:
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@@
 		)
 	)
-	(text "Pro		RFM9x	\nMini\n-----------\nVCC	 	3.3V\nGND	 	GND	 \nD2		DIO0	 \nD3		DIO1\nD7		DIO2	 \nD6		DIO5\nD5		RESET	 	 \nD10-SS	NSS	 \nMOSI	MOSI	 \nMISO	MISO	 \nCLK		SCK"
+	(text "Pro			RFM9x	\nMini\n-----------\nVCC	 		3.3V\nGND	 		GND	 \nD2			DIO0	 \nD3			DIO1\nD7			DIO2	 \nD6			DIO5\nD5			RESET	 	 \nD10-SS		NSS	 \nD11-MOSI	MOSI	 \nD12-MISO	MISO	 \nD13-CLK		SCK"
 		(exclude_from_sim no)
 		(at 179.832 138.43 0)

Commit message: Small fixes
Other:
- note added: "+3.3V"
- note added: "RAW"
- moved on the sheet: JP1, R1
Changed lines of the file:
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@@
 	)
 	(junction
-		(at 219.71 125.73)
+		(at 219.71 123.825)
 		(diameter 0)
 		(color 0 0 0 0)
@@
 	(wire
 		(pts
-			(xy 219.71 127) (xy 219.71 125.73)
+			(xy 219.71 125.095) (xy 219.71 123.825)
 		)
 		(stroke
@@
 	(wire
 		(pts
-			(xy 219.71 125.73) (xy 219.71 121.92)
+			(xy 219.71 123.825) (xy 219.71 120.015)
 		)
 		(stroke
@@
 	(wire
 		(pts
+			(xy 227.33 127.635) (xy 227.33 129.54)
+		)
+		(stroke
+			(width 0)
+			(type default)
+		)
+	)
+	(wire
+		(pts
 			(xy 224.79 44.45) (xy 215.9 44.45)
 		)
@@
 	(wire
 		(pts
-			(xy 232.41 125.73) (xy 234.95 125.73)
+			(xy 232.41 123.825) (xy 234.95 123.825)
 		)
 		(stroke
@@
 	(wire
 		(pts
+			(xy 219.71 132.715) (xy 219.71 134.62)
+		)
+		(stroke
+			(width 0)
+			(type default)
+		)
+	)
+	(wire
+		(pts
 			(xy 106.68 120.65) (xy 114.3 120.65)
 		)
@@
 	(wire
 		(pts
-			(xy 222.25 125.73) (xy 219.71 125.73)
+			(xy 222.25 123.825) (xy 219.71 123.825)
 		)
 		(stroke
@@
 	(wire
 		(pts
-			(xy 234.95 121.92) (xy 234.95 125.73)
+			(xy 234.95 120.015) (xy 234.95 123.825)
 		)
 		(stroke
@@
 		)
 	)
+	(text "+3.3V"
+		(exclude_from_sim no)
+		(at 190.5 53.975 0)
+		(effects
+			(font
+				(size 2 2)
+				(thickness 0.4)
+				(bold yes)
+			)
+		)
+	)
+	(text "RAW"
+		(exclude_from_sim no)
+		(at 189.23 48.26 0)
+		(effects
+			(font
+				(size 2 2)
+				(thickness 0.4)
+				(bold yes)
+			)
+		)
+	)
 	(text "Pro			RFM9x	\nMini\n-----------\nVCC	 		3.3V\nGND	 		GND	 \nD2			DIO0	 \nD3			DIO1\nD7			DIO2	 \nD6			DIO5\nD5			RESET	 	 \nD10-SS		NSS	 \nD11-MOSI	MOSI	 \nD12-MISO	MISO	 \nD13-CLK		SCK"
 		(exclude_from_sim no)
@@
 		)
 	)
+	(text "RAW"
+		(exclude_from_sim no)
+		(at 240.665 118.11 0)
+		(effects
+			(font
+				(size 2 2)
+				(thickness 0.4)
+				(bold yes)
+			)
+		)
+	)
 	(global_label "RX1"
 		(shape input)
@@
 	(symbol
 		(lib_id "ProMini-Node-v1.0-50x50-rescue:SolderJumper_3_Open-Jumper")
-		(at 227.33 125.73 0)
+		(at 227.33 123.825 0)
 		(unit 1)
 		(exclude_from_sim no)
@@
 		(dnp no)
 		(property "Reference" "JP1"
-			(at 227.33 123.444 0)
+			(at 227.33 121.539 0)
 			(effects
 				(font
@@
 		)
 		(property "Value" "Voltage Measurement"
-			(at 239.776 127.508 0)
+			(at 239.776 125.603 0)
 			(effects
 				(font
@@
 		)
 		(property "Footprint" "Jumper:SolderJumper-3_P1.3mm_Open_RoundedPad1.0x1.5mm_NumberLabels"
-			(at 227.33 125.73 0)
+			(at 227.33 123.825 0)
 			(effects
 				(font
@@
 		)
 		(property "Datasheet" "~"
-			(at 227.33 125.73 0)
+			(at 227.33 123.825 0)
 			(effects
 				(font
@@
 		)
 		(property "Description" ""
-			(at 227.33 125.73 0)
+			(at 227.33 123.825 0)
 			(effects
 				(font
@@
 	(symbol
 		(lib_id "Device:R")
-		(at 219.71 130.81 0)
+		(at 219.71 128.905 0)
 		(unit 1)
 		(exclude_from_sim no)
@@
 		(dnp no)
 		(property "Reference" "R1"
-			(at 213.106 128.778 0)
+			(at 213.106 126.873 0)
 			(effects
 				(font
@@
 		)
 		(property "Value" "100K"
-			(at 212.852 131.064 0)
+			(at 212.852 129.159 0)
 			(effects
 				(font
@@
 		)
 		(property "Footprint" "Resistor_SMD:R_0805_2012Metric_Pad1.15x1.40mm_HandSolder"
-			(at 217.932 130.81 90)
+			(at 217.932 128.905 90)
 			(effects
 				(font
@@
 		)
 		(property "Datasheet" "~"
-			(at 219.71 130.81 0)
+			(at 219.71 128.905 0)
 			(effects
 				(font
@@
 		)
 		(property "Description" ""
-			(at 219.71 130.81 0)
+			(at 219.71 128.905 0)
 			(effects
 				(font
@@
 	(symbol
 		(lib_id "ProMini-Node-v1.0-50x50-rescue:+3.3V-power")
-		(at 219.71 121.92 0)
+		(at 219.71 120.015 0)
 		(unit 1)
 		(exclude_from_sim no)
@@
 		(dnp no)
 		(property "Reference" "#PWR0106"
-			(at 219.71 125.73 0)
+			(at 219.71 123.825 0)
 			(effects
 				(font
@@
 		)
 		(property "Value" "+3V3"
-			(at 219.71 118.364 0)
+			(at 219.71 116.459 0)
 			(effects
 				(font
@@
 		)
 		(property "Footprint" ""
-			(at 219.71 121.92 0)
+			(at 219.71 120.015 0)
 			(effects
 				(font
@@
 		)
 		(property "Datasheet" ""
-			(at 219.71 121.92 0)
+			(at 219.71 120.015 0)
 			(effects
 				(font
@@
 		)
 		(property "Description" ""
-			(at 219.71 121.92 0)
+			(at 219.71 120.015 0)
 			(effects
 				(font
@@
 	(symbol
 		(lib_id "power:VCC")
-		(at 234.95 121.92 0)
+		(at 234.95 120.015 0)
 		(unit 1)
 		(exclude_from_sim no)
@@
 		(dnp no)
 		(property "Reference" "#PWR0108"
-			(at 234.95 125.73 0)
+			(at 234.95 123.825 0)
 			(effects
 				(font
@@
 		)
 		(property "Value" "VCC"
-			(at 235.3818 117.5258 0)
+			(at 235.3818 115.6208 0)
 			(effects
 				(font
@@
 		)
 		(property "Footprint" ""
-			(at 234.95 121.92 0)
+			(at 234.95 120.015 0)
 			(effects
 				(font
@@
 		)
 		(property "Datasheet" ""
-			(at 234.95 121.92 0)
+			(at 234.95 120.015 0)
 			(effects
 				(font
@@
 		)
 		(property "Description" ""
-			(at 234.95 121.92 0)
+			(at 234.95 120.015 0)
 			(effects
 				(font
